File: PCB/BQ76920.kicad_sch (KiCad schematic)
At the start: 81 parts, among them CN6 WAFER-SH1.0-6PWB, Q1 CSD13381F4, Q10 TP0610K-T1-GE3, Q2 CSD13381F4, Q3 CSD13381F4, Q4 CSD13381F4, Q5 CSD13381F4, Q6 BSC0702LS, Q7 BSC0702LS, Q8 BSC0702LS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

Commit message: xudangling initial commit
Parts:
- renumbered C20 to C10, C28 to C11, C16 to C12, C9 to C13, C10 to C14, C24 to C15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
Other:
- moved on the sheet: C10, C11, C12, C9, D4, D5, H5, H6, H7, H8, L2, R11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
