File: PCB/CawBMS.kicad_pcb (KiCad board)
At the start: 4 copper layers, 53.5 x 38 mm, 132 parts, among them CN1 SWD, CN2 I2C, CN3 SPI, CN4 USART, CN5 SWD, CN6 WAFER-SH1.0-6PWB, Q1 CSD13381F4, Q10 TP0610K-T1-GE3, Q2 CSD13381F4, Q3 CSD13381F4, Q4 CSD13381F4, Q5 CSD13381F4, Q6 BSC0702LS, Q7 BSC0702LS, Q8 BSC0702LS, Q9 BSC0702LS, SW1 B3U-1000P, SW2 B3U-1000P, SW3 B3U-1000P, U1 STM32F103CBTx, U2 TCAN1044DRBRQ1, U3 TPS61240DRVR, U4 BQ7692003PW, U5 CAN, X1 Crystal_16MHz_15pF_3P

Commit message: xudangling initial commit
Parts:
- removed R40: 1M, Resistor_SMD:R_0402_1005Metric_Pad0.72x0.64mm_HandSolder
- removed REF**: OSHW-Logo2_9.8x8mm_SilkScreen, Symbol:OSHW-Logo2_9.8x8mm_SilkScreen
- removed U5: CAN, Rick_Connector:CONN-SMD_2P-P1.00_XUNPU_WAFER-SH1.0-2PWB
- added CN7: WAFER-SH1.0-6PWB, Rick_Connector:CONN-SMD_6P-P1.00_XUNPU_WAFER-SH1.0-6PWB, F.Cu at (64.5, 39.5)
- added R11: 0, Resistor_SMD:R_0402_1005Metric_Pad0.72x0.64mm_HandSolder, F.Cu at (121.5, 35.0)
- C10: value 0.22uF -> 4.7uF
- C11, C9: value 0.22uF -> 0.1uF; footprint Capacitor_SMD:C_0402_1005Metric_Pad0.74x0.62mm_HandSolder -> Capacitor_SMD:C_0603_1608Metric_Pad1.08x0.95mm_HandSolder
- C12: value 0.22uF -> 2.2uF
- C15: value 4.7uF -> 470pF
- C16: value 2.2uF -> 1uF
- C17: value 1uF -> 0.22uF
- C18: value 1uF -> 4.7uF
- C19: value 10uF -> 1uF; footprint Capacitor_SMD:C_0603_1608Metric_Pad1.08x0.95mm_HandSolder -> Capacitor_SMD:C_0402_1005Metric_Pad0.74x0.62mm_HandSolder
- C20: value 4.7uF -> 10uF; footprint Capacitor_SMD:C_0402_1005Metric_Pad0.74x0.62mm_HandSolder -> Capacitor_SMD:C_0603_1608Metric_Pad1.08x0.95mm_HandSolder
- C21, C22: value 0.1uF -> 0.22uF
- C24: value 470pF -> 0.1uF
- C25: footprint Capacitor_SMD:C_0603_1608Metric_Pad1.08x0.95mm_HandSolder -> Capacitor_SMD:C_0402_1005Metric_Pad0.74x0.62mm_HandSolder
- C26: value 0.1uF -> 0.22uF; footprint Capacitor_SMD:C_0603_1608Metric_Pad1.08x0.95mm_HandSolder -> Capacitor_SMD:C_0402_1005Metric_Pad0.74x0.62mm_HandSolder
- CN1: value SWD -> CAN; footprint Rick_Connector:CONN-SMD_4P-P1.00_WAFER-SH1.0-4PWB -> Rick_Connector:CONN-SMD_2P-P1.00_XUNPU_WAFER-SH1.0-2PWB
- CN2: value I2C -> SWD
- CN3: value SPI -> I2C; footprint Rick_Connector:CONN-SMD_6P-P1.00_XUNPU_WAFER-SH1.0-6PWB -> Rick_Connector:CONN-SMD_4P-P1.00_WAFER-SH1.0-4PWB
- CN4: value USART -> SPI; footprint Rick_Connector:CONN-SMD_4P-P1.00_WAFER-SH1.0-4PWB -> Rick_Connector:CONN-SMD_6P-P1.00_XUNPU_WAFER-SH1.0-6PWB
- CN5: value SWD -> USART
- CN6: value WAFER-SH1.0-6PWB -> POWER; footprint Rick_Connector:CONN-SMD_6P-P1.00_XUNPU_WAFER-SH1.0-6PWB -> Rick_Connector:CONN-SMD_4P-P1.00_WAFER-SH1.0-4PWB
- D10: value D_200V -> D_Zener_5.6V; footprint Diode_SMD:D_SMA_Handsoldering -> Diode_SMD:D_SOD-523
- D11: value D_100V -> D_Zener_16V; footprint Diode_SMD:D_SOD-323_HandSoldering -> Diode_SMD:D_SOD-523
- D12: value D_Zener_16V -> D_Zener_5.6V
- D4: value D_Zener_5.6V -> TVS_24V; footprint Diode_SMD:D_SOD-523 -> Diode_SMD:D_SMA_Handsoldering
- D5: value D_Zener_5.6V -> D_200V; footprint Diode_SMD:D_SOD-523 -> Diode_SMD:D_SMA_Handsoldering
- D9: value TVS_24V -> D_100V; footprint Diode_SMD:D_SMA_Handsoldering -> Diode_SMD:D_SOD-323_HandSoldering
- H6: value B- -> P+
- H7: value P+ -> B-
- Q10: value TP0610K-T1-GE3 -> BSC0702LS; footprint Package_TO_SOT_SMD:SOT-23 -> Rick_MOSFET:BSC0702LS_PG-TDSON-8_L5.0-W6.0-P1.27-BL-EP
- Q4: value CSD13381F4 -> TP0610K-T1-GE3; footprint Rick_MOSFET:CSD13381F4_PICOSTAR-3_L1.0-W0.6-P0.40-S0.65-BL-1 -> Package_TO_SOT_SMD:SOT-23
- Q6: value BSC0702LS -> CSD13381F4; footprint Rick_MOSFET:BSC0702LS_PG-TDSON-8_L5.0-W6.0-P1.27-BL-EP -> Rick_MOSFET:CSD13381F4_PICOSTAR-3_L1.0-W0.6-P0.40-S0.65-BL-1
- R1: value 10k -> 120
- R12, R15: value 28.7 -> 100
- R14: value 28.7 -> 10k
- R17: value 100 -> 499k
- R19, R27, R31: value 100 -> 10k
- R20: value 10k -> NTC 10k
- R22, R26: value 10k -> 28.7
- R28: value NTC 10k -> 1M
- R29: value 10k -> 100
- R3: value 0 -> 10k
- R30: value 100 -> 28.7
- R32: value 0.0015 -> 1M; footprint Resistor_SMD:R_2512_6332Metric_Pad1.40x3.35mm_HandSolder -> Resistor_SMD:R_0402_1005Metric_Pad0.72x0.64mm_HandSolder
- R33, R34: value 0.0015 -> 100; footprint Resistor_SMD:R_2512_6332Metric_Pad1.40x3.35mm_HandSolder -> Resistor_SMD:R_0402_1005Metric_Pad0.72x0.64mm_HandSolder
- R35: value 100 -> 1M
- R36, R39: value 1M -> 0.0015; footprint Resistor_SMD:R_0402_1005Metric_Pad0.72x0.64mm_HandSolder -> Resistor_SMD:R_2512_6332Metric_Pad1.40x3.35mm_HandSolder
- R37: value 0 -> 100
- R38: value 499k -> 0.0015; footprint Resistor_SMD:R_0402_1005Metric_Pad0.72x0.64mm_HandSolder -> Resistor_SMD:R_2512_6332Metric_Pad1.40x3.35mm_HandSolder
- R6: value 120 -> 10k
- R7: value 510 -> 0
- R8: value 10k -> 510
- U1: value STM32F103CBTx -> SIT1051AT/3; footprint Package_QFP:LQFP-48_7x7mm_P0.5mm -> Rick_CAN:ISO1044BDR_SOP-8
- U2: value TCAN1044DRBRQ1 -> STM32F103C_8-B_Tx; footprint Rick_CAN:TCAN1044DRBRQ1_DFN-8_L3.0-W3.0-P0.65-TL-EP2.4 -> Package_QFP:LQFP-48_7x7mm_P0.5mm
- moved C1 63.7 mm to (107.6, 47.0)
- moved C10 63.7 mm to (92.4, 46.8)
- moved C11 63.7 mm to (92.4, 49.8)
- moved C15 63.7 mm to (105.0, 56.7)
- moved C24 63.7 mm to (102.1, 49.4)
- moved C26 63.7 mm to (105.4, 66.5)
- moved C4 63.7 mm to (107.6, 45.8)
- moved C5 63.7 mm to (120.4, 49.0)
- moved C6 63.7 mm to (105.0, 54.2)
- moved C8 63.7 mm to (105.0, 51.7)
- moved CN5 63.7 mm to (125.8, 48.5)
- moved CN6 63.7 mm to (78.8, 49.8)
- moved L4 63.7 mm to (99.8, 66.5)
- moved L5 63.7 mm to (111.5, 66.5)
- moved Q3 63.7 mm to (86.1, 49.8)
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Connections:
- C1 pad 1: +3.3V -> +5V
- C10 pad 1: /BQ76920/VC4 -> +5V
- C10 pad 2: /BQ76920/VC3 -> GND
- C11 pad 1: /BQ76920/VC3 -> Net-(C11-Pad1)
- C11 pad 2: /BQ76920/VC2 -> PACK-
- C12 pad 1: /BQ76920/VC2 -> +3.3V
- C12 pad 2: /BQ76920/VC1 -> GND
- C13 pad 1: /BQ76920/VC1 -> /BQ76920/VC5
- C13 pad 2: /BQ76920/VC0 -> /BQ76920/VC4
- C14 pad 1: /BQ76920/VC0 -> /BQ76920/VC4
- C14 pad 2: GND -> /BQ76920/VC3
- C15 pad 1: +3.3V -> /ALERT
- C16 pad 1: +3.3V -> GND
- C16 pad 2: GND -> Net-(U4-CAP1)
- C17 pad 1: /BQ76920/BAT -> /BQ76920/VC3
- C17 pad 2: GND -> /BQ76920/VC2
- C18 pad 1: GND -> +3.3V
- C18 pad 2: Net-(U4-CAP1) -> GND
- C19 pad 1: Net-(U4-BAT) -> /BQ76920/BAT
- C20 pad 1: +5V -> Net-(U4-BAT)
- C21 pad 1: GND -> /BQ76920/VC2
- C21 pad 2: /BQ76920/SRP -> /BQ76920/VC1
- C22 pad 1: /BQ76920/SRP -> /BQ76920/VC1
- C22 pad 2: /BQ76920/SRN -> /BQ76920/VC0
- C23 pad 1: /BQ76920/SRN -> GND
- C23 pad 2: GND -> /BQ76920/SRP
- C24 pad 1: /ALERT -> /BQ76920/SRP
- C24 pad 2: GND -> /BQ76920/SRN
- C25 pad 1: Net-(C25-Pad1) -> /BQ76920/SRN
- C25 pad 2: Net-(C25-Pad2) -> GND
- C26 pad 1: Net-(C25-Pad2) -> /BQ76920/VC0
- C26 pad 2: PACK- -> GND
- C27 pad 1: PACK+ -> Net-(C27-Pad1)
- C3 pad 1: +3.3V -> /RESET
- C5 pad 1: +5V -> +3.3V
- C6 pad 1: +3.3VA -> +3.3V
- C8 pad 1: /RESET -> +3.3VA
- C9 pad 1: /BQ76920/VC5 -> PACK+
- C9 pad 2: /BQ76920/VC4 -> Net-(C11-Pad1)
- CN1 pad 1: GND -> /CAN_N
- CN1 pad 2: GND -> /CAN_P
- CN1 pad 3: +3.3V -> unconnected-(CN1-Pad3)
- CN1 pad 4: +5V -> unconnected-(CN1-Pad4)
- CN2 pad 1: /I2C2_SDA -> /SWDIO
- CN2 pad 2: /I2C2_SCL -> /SWCLK
- CN3 pad 1: /SPI1_NSS -> /I2C2_SDA
- CN3 pad 2: /SPI1_SCK -> /I2C2_SCL
- CN3 pad 3: /SPI1_MISO -> GND
- CN3 pad 4: /SPI1_MOSI -> +3.3V
- CN3 pad 5: GND -> unconnected-(CN3-Pad5)
- CN3 pad 6: +3.3V -> unconnected-(CN3-Pad6)
- CN4 pad 1: /USART1_TX -> /SPI1_NSS
- CN4 pad 2: /USART1_RX -> /SPI1_SCK
- CN4 pad 3: GND -> /SPI1_MISO
- CN4 pad 4: +3.3V -> /SPI1_MOSI
- CN4 pad 5: unconnected-(CN4-Pad5) -> GND
- CN4 pad 6: unconnected-(CN4-Pad6) -> +3.3V
- CN5 pad 1: /SWDIO -> /USART1_TX
- CN5 pad 2: /SWCLK -> /USART1_RX
- CN6 pad 1: /BQ76920/BAT -> GND
- CN6 pad 2: Net-(D4-A) -> GND
- CN6 pad 3: Net-(D5-A) -> +3.3V
- CN6 pad 4: Net-(D6-A) -> +5V
- CN6 pad 5: Net-(D7-A) -> unconnected-(CN6-Pad5)
- CN6 pad 6: Net-(D8-A) -> unconnected-(CN6-Pad6)
- D10 pad 1: PACK+ -> Net-(D10-K)
- D10 pad 2: PACK- -> Net-(D10-A)
- D11 pad 2: Net-(D11-A) -> PACK-
- D12 pad 1: Net-(D11-K) -> Net-(D12-K)
- D12 pad 2: PACK- -> Net-(D12-A)
- D4 pad 1: Net-(D4-K) -> -BATT
- D4 pad 2: Net-(D4-A) -> PACK+
- D5 pad 1: Net-(D5-K) -> PACK+
- D5 pad 2: Net-(D5-A) -> PACK-
- D9 pad 1: -BATT -> Net-(D11-K)
- D9 pad 2: PACK+ -> Net-(D9-A)
- H6 pad 1: -BATT -> PACK+
- H7 pad 1: PACK+ -> -BATT
- L3 pad 2: Net-(Q7-G) -> Net-(Q9-G)
- L4 pad 2: Net-(Q6-G) -> Net-(Q7-G)
- L6 pad 2: Net-(Q9-G) -> Net-(Q10-G)
- Q1 pad 1: Net-(D4-K) -> Net-(D6-K)
- Q1 pad 2: Net-(D4-A) -> Net-(D6-A)
- Q10 pad 1: GND -> PACK-
- Q10 pad 2: /BQ76920/CHG -> PACK-
- Q10 pad 3: Net-(D11-A) -> PACK-
- Q2 pad 1: Net-(D5-K) -> Net-(D7-K)
- Q2 pad 2: Net-(D5-A) -> Net-(D7-A)
- Q3 pad 1: Net-(D6-K) -> Net-(D8-K)
- Q3 pad 2: Net-(D6-A) -> Net-(D8-A)
- Q4 pad 1: Net-(D7-K) -> GND
- Q4 pad 2: Net-(D7-A) -> /BQ76920/CHG
- Q4 pad 3: Net-(Q4-D) -> Net-(D9-A)
- Q5 pad 1: Net-(D8-K) -> Net-(D10-K)
- Q5 pad 2: Net-(D8-A) -> Net-(D10-A)
- Q6 pad 1: Net-(C25-Pad1) -> Net-(D12-K)
- Q6 pad 2: Net-(C25-Pad1) -> Net-(D12-A)
- Q6 pad 3: Net-(C25-Pad1) -> Net-(Q6-D)
- Q7 pad 1: Net-(C25-Pad1) -> Net-(C27-Pad1)
- Q7 pad 2: Net-(C25-Pad1) -> Net-(C27-Pad1)
- Q7 pad 3: Net-(C25-Pad1) -> Net-(C27-Pad1)
- Q7 pad 5: Net-(Q6-D-Pad5) -> Net-(Q10-D-Pad5)
- Q7 pad 6: Net-(Q6-D-Pad5) -> Net-(Q10-D-Pad5)
- Q7 pad 7: Net-(Q6-D-Pad5) -> Net-(Q10-D-Pad5)
- Q7 pad 8: Net-(Q6-D-Pad5) -> Net-(Q10-D-Pad5)
- Q8 pad 5: Net-(Q6-D-Pad5) -> Net-(Q10-D-Pad5)
- Q8 pad 6: Net-(Q6-D-Pad5) -> Net-(Q10-D-Pad5)
- Q8 pad 7: Net-(Q6-D-Pad5) -> Net-(Q10-D-Pad5)
- Q8 pad 8: Net-(Q6-D-Pad5) -> Net-(Q10-D-Pad5)
- Q9 pad 1: PACK- -> Net-(C27-Pad1)
- Q9 pad 2: PACK- -> Net-(C27-Pad1)
- Q9 pad 3: PACK- -> Net-(C27-Pad1)
- Q9 pad 5: Net-(Q6-D-Pad5) -> Net-(Q10-D-Pad5)
- Q9 pad 6: Net-(Q6-D-Pad5) -> Net-(Q10-D-Pad5)
- Q9 pad 7: Net-(Q6-D-Pad5) -> Net-(Q10-D-Pad5)
- Q9 pad 8: Net-(Q6-D-Pad5) -> Net-(Q10-D-Pad5)
- R1 pad 1: GND -> /CAN_N
- R1 pad 2: Net-(U1-PB2) -> /CAN_P
- R12 pad 2: Net-(Q1-D) -> /BQ76920/VC5
- R13 pad 1: Net-(D4-A) -> /BQ76920/BAT
- R13 pad 2: Net-(Q2-D) -> Net-(Q1-D)
- R14 pad 1: Net-(D5-A) -> Net-(D6-K)
- R14 pad 2: Net-(Q3-D) -> /BQ76920/VC4
- R15 pad 2: Net-(Q4-D) -> /BQ76920/VC4
- R16 pad 1: Net-(D7-A) -> Net-(D6-A)
- R16 pad 2: Net-(Q5-D) -> Net-(Q2-D)
- R17 pad 1: /BQ76920/BAT -> GND
- R17 pad 2: /BQ76920/VC5 -> /ALERT
- R18 pad 1: Net-(D4-K) -> Net-(D7-K)
- R18 pad 2: /BQ76920/VC4 -> /BQ76920/VC3
- R19 pad 1: Net-(D4-A) -> Net-(R19-Pad1)
- R19 pad 2: /BQ76920/VC4 -> Net-(U4-TS1)
- R2 pad 2: Net-(U1-BOOT0) -> Net-(U2-BOOT0)
- R20 pad 1: Net-(D5-K) -> GND
- R20 pad 2: /BQ76920/VC3 -> Net-(U4-TS1)
- R21 pad 1: Net-(D5-A) -> Net-(D7-A)
- R22 pad 1: Net-(D6-K) -> Net-(D7-A)
- R22 pad 2: /BQ76920/VC2 -> Net-(Q3-D)
- R23 pad 1: Net-(D6-A) -> /BQ76920/BAT
- R23 pad 2: /BQ76920/VC2 -> Net-(U4-BAT)
- R24 pad 1: Net-(D7-K) -> Net-(D8-K)
- R24 pad 2: /BQ76920/VC1 -> /BQ76920/VC2
- R25 pad 1: Net-(D7-A) -> Net-(D8-A)
- R25 pad 2: /BQ76920/VC1 -> /BQ76920/VC2
- R26 pad 1: Net-(D8-K) -> Net-(D8-A)
- R26 pad 2: /BQ76920/VC0 -> Net-(Q5-D)
- R27 pad 1: Net-(D8-A) -> Net-(D10-K)
- R27 pad 2: /BQ76920/VC0 -> /BQ76920/VC1
- R28 pad 1: GND -> Net-(D11-K)
- R28 pad 2: Net-(U4-TS1) -> Net-(D9-A)
- R29 pad 1: Net-(R29-Pad1) -> Net-(D10-A)
- R29 pad 2: Net-(U4-TS1) -> /BQ76920/VC1
- R3 pad 1: Net-(U1-VSSA) -> +3.3V
- R3 pad 2: GND -> /I2C1_SCL
- R30 pad 1: /BQ76920/BAT -> Net-(D10-A)
- R30 pad 2: Net-(U4-BAT) -> Net-(Q6-D)
- R31 pad 1: -BATT -> Net-(D12-K)
- R31 pad 2: /BQ76920/SRP -> /BQ76920/VC0
- R32 pad 1: -BATT -> PACK-
- R32 pad 2: Net-(C25-Pad1) -> Net-(D11-K)
- R33 pad 2: Net-(C25-Pad1) -> /BQ76920/SRP
- R34 pad 1: -BATT -> Net-(C27-Pad1)
- R34 pad 2: Net-(C25-Pad1) -> /BQ76920/SRN
- R35 pad 1: Net-(C25-Pad1) -> Net-(C27-Pad1)
- R35 pad 2: /BQ76920/SRN -> /BQ76920/DSG
- R36 pad 1: Net-(C25-Pad1) -> -BATT
- R36 pad 2: /BQ76920/DSG -> Net-(C27-Pad1)
- R37 pad 1: -BATT -> Net-(D12-A)
- R37 pad 2: GND -> /BQ76920/VC0
- R38 pad 1: GND -> -BATT
- R38 pad 2: /ALERT -> Net-(C27-Pad1)
- R39 pad 1: Net-(D11-K) -> -BATT
- R39 pad 2: Net-(D11-A) -> Net-(C27-Pad1)
- R4 pad 2: /I2C1_SCL -> /I2C1_SDA
- R5 pad 1: +3.3V -> GND
- R5 pad 2: /I2C1_SDA -> Net-(U2-PB2)
- R6 pad 1: /CAN_N -> +3.3V
- R6 pad 2: /CAN_P -> /RESET
- R7 pad 1: Net-(D1-K) -> Net-(U2-VSSA)
- R7 pad 2: /LED_A -> GND
- R8 pad 1: +3.3V -> Net-(D1-K)
- R8 pad 2: /RESET -> /LED_A
- SW3 pad 2: Net-(R29-Pad1) -> Net-(R19-Pad1)
- U1 pad 1: +3.3V -> /CAN_TX
- U1 pad 2: /ALERT -> GND
- U1 pad 3: /LED_A -> +5V
- U1 pad 4: /LED_B -> /CAN_RX
- U1 pad 5: /HSE_IN -> +3.3V
- U1 pad 6: /HSE_OUT -> /CAN_N
- U1 pad 7: /RESET -> /CAN_P
- U1 pad 8: Net-(U1-VSSA) -> /CAN_S
- U2 pad 1: /CAN_TX -> +3.3V
- U2 pad 2: GND -> /ALERT
- U2 pad 3: +5V -> /LED_A
- U2 pad 4: /CAN_RX -> /LED_B
- U2 pad 5: +3.3V -> /HSE_IN
- U2 pad 6: /CAN_N -> /HSE_OUT
- U2 pad 7: /CAN_P -> /RESET
- U2 pad 8: /CAN_STB -> Net-(U2-VSSA)
- U2 pad 9: GND -> +3.3VA
Routing:
- net (no net): track 0.00 -> 83.9 mm, vias 0 -> 19
- net Net-(R29-Pad1): track 26.1 -> 0.00 mm
- net Net-(C25-Pad1): track 16.4 -> 0.00 mm, vias 17 -> 0
- net Net-(D4-A): track 13.1 -> 0.00 mm
- net Net-(D5-A): track 12.8 -> 0.00 mm
- net /I2C2_SDA: track 16.5 -> 26.3 mm
- net /I2C2_SCL: track 16.9 -> 26.2 mm
- net /CAN_STB: track 7.70 -> 0.00 mm, vias 2 -> 0
- net unconnected-(U2-PB0-Pad18): track 0.00 -> 7.70 mm, vias 0 -> 2
- net /SPI1_MOSI: track 8.68 -> 1.33 mm
- net unconnected-(U2-PA6-Pad16): track 0.00 -> 6.83 mm, vias 0 -> 2
- net /CAN_TX: track 6.83 -> 0.00 mm, vias 2 -> 0
- net PACK-: track 8.30 -> 2.28 mm, vias 17 -> 15
- net Net-(Q7-G): track 2.25 -> 8.21 mm
- net Net-(Q6-G): track 5.95 -> 0.00 mm
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- removed copper zone on In2.Cu, net +3.3V
- removed copper zone on B.Cu, net -BATT
- removed copper zone on F.Cu, net -BATT
- removed copper zone on In1.Cu, net -BATT
- removed copper zone on In2.Cu, net -BATT
- removed copper zone on In1.Cu, net GND
- removed copper zone on B.Cu, net Net-(C25-Pad1)
- removed copper zone on F.Cu, net Net-(C25-Pad1)
- removed copper zone on In1.Cu, net Net-(C25-Pad1)
- removed copper zone on In2.Cu, net Net-(C25-Pad1)
- removed copper zone on F.Cu, net Net-(Q6-D-Pad5)
- removed copper zone on In1.Cu, net Net-(Q6-D-Pad5)
- removed copper zone on B.Cu, net PACK+
- removed copper zone on F.Cu, net PACK+
- removed copper zone on In1.Cu, net PACK+
- removed copper zone on In2.Cu, net PACK+
- removed copper zone on B.Cu, net PACK-
- removed copper zone on F.Cu, net PACK-
- removed copper zone on In1.Cu, net PACK-
- removed copper zone on In2.Cu, net PACK-
